File: pcb/board/pro/Wonkle.kicad_sch (KiCad schematic)
At the start: 21 parts, among them J1 USB_C_Receptacle_USB2.0_16P, J2 Conn_01x04_Pin, SW1 EVQQ2B03W, SW2 EVQQ2B03W, U229 STM32F429IGT6, U231 TPS62152

Commit message: Update PCB with HSE oscillator, Footprint Mismatch fix and Rename project files to Wonkle (#36)
Parts:
- added C255, C256: 10p, Capacitor_SMD:C_0402_1005Metric, symbol Device:C
- added R26: 2k, Resistor_SMD:R_0402_1005Metric, symbol Device:R
- added Y1: Crystal, Crystal:Crystal_SMD_5032-2Pin_5.0x3.2mm, symbol Device:Crystal
Connections:
- net GND: now also J1.SH (SHIELD), C255.1, C256.2; no longer J1.S1 (SHIELD)
- net at U229.29 (PH0): now also C255.2, Y1.2
- net at U229.30 (PH1): now also R26.1
- new net: C256.1, R26.2, Y1.1
- no-connect marks 119 -> 117
Other:
- note added: "USB HSE"
- title: Pompyboard Prototype -> Wonkle Prototype
- moved on the sheet: C20, C21, C22, C251, C252, C253, C254, D1, J1, J2, L1, R20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
